File: MCU.kicad_sch (KiCad schematic)
At the start: 28 parts, among them J10 Conn_02x03_Odd_Even, J3 Conn_01x03, J4 Conn_01x04, U2 STM32G431CBUx, Y1 24MHz, 9pF

Commit message: WIP
Connections:
- net +3.3V is gone; now on net +3V3: L1.2
Changed lines of the file:
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@@
 			)
 		)
-		(property "Value" "+3.3V"
+		(property "Value" "+3V3"
 			(at 194.31 58.0969 0)
 			(effects

Commit message: Routing
Connections:
- net USB_MCU_D-: now reaches R4.1, U2.33 (PA11)
- net USB_MCU_D+: now reaches R5.1, U2.34 (PA12)
Other:
- sheet Power ports: added USB_D+, USB_D-; removed none
Changed lines of the file:
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@@
 	(wire
 		(pts
+			(xy 63.5 43.18) (xy 76.2 43.18)
+		)
+		(stroke
+			(width 0)
+			(type default)
+		)
+	)
+	(wire
+		(pts
 			(xy 138.43 72.39) (xy 138.43 73.66)
 		)
@@
 	(wire
 		(pts
+			(xy 63.5 45.72) (xy 76.2 45.72)
+		)
+		(stroke
+			(width 0)
+			(type default)
+		)
+	)
+	(wire
+		(pts
 			(xy 158.75 101.6) (xy 168.91 101.6)
 		)
@@
 		)
 	)
+	(label "USB_MCU_D+"
+		(at 173.99 111.76 180)
+		(effects
+			(font
+				(size 1.27 1.27)
+			)
+			(justify right bottom)
+		)
+	)
 	(label "opamp3_vinp"
 		(at 109.22 152.4 0)
@@
 		)
 	)
+	(label "USB_D+"
+		(at 76.2 43.18 180)
+		(effects
+			(font
+				(size 1.27 1.27)
+			)
+			(justify right bottom)
+		)
+	)
 	(label "dac1_out2"
 		(at 173.99 93.98 180)
@@
 		)
 	)
+	(label "USB_MCU_D-"
+		(at 173.99 109.22 180)
+		(effects
+			(font
+				(size 1.27 1.27)
+			)
+			(justify right bottom)
+		)
+	)
 	(label "SPI3_MISO"
 		(at 111.76 106.68 0)
@@
 		)
 	)
+	(label "USB_D-"
+		(at 76.2 45.72 180)
+		(effects
+			(font
+				(size 1.27 1.27)
+			)
+			(justify right bottom)
+		)
+	)
 	(label "VREF+"
 		(at 114.3 81.28 0)
@@
 			(effects
 				(font
+					(size 1.27 1.27)
+				)
+				(justify right)
+			)
+		)
+		(pin "USB_D+" input
+			(at 63.5 43.18 0)
+			(effects
+				(font
+					(size 1.27 1.27)
+				)
+				(justify right)
+			)
+		)
+		(pin "USB_D-" input
+			(at 63.5 45.72 0)
+			(effects
+				(font

Commit message: Preliminary routing done
Connections:
- net SPI3_MISO: now also J10.1 (Pin_1); no longer J10.5 (Pin_5)
- net SPI3_MOSI: now also J10.5 (Pin_5); no longer J10.3 (Pin_3)
- net SPI3_SCK: now also J10.3 (Pin_3); no longer J10.1 (Pin_1)
- net opamp2_vinp: now also J4.3 (Pin_3); no longer J4.2 (Pin_2)
- net opamp3_vinp: now also J4.2 (Pin_2); no longer J4.3 (Pin_3)
