File: opamp_ldc.kicad_sch (KiCad schematic)
At the start: 14 parts, among them J8 Conn_Coaxial, J9 Conn_Coaxial, U5 TPH2502-SR

Commit message: Preliminary routing done
Changed lines of the file:
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@@
 					(size 1.27 1.27)
 				)
+				(hide yes)
 			)
 		)
@@
 					(size 1.27 1.27)
 				)
-			)
-		)
+				(hide yes)
+			)
+		)
